Commit message: add wheels

File: Project2/catkin_ws/src/my_robot/urdf/my_robot.xacro (robot description, xacro)
@@ -54,3 +54,59 @@
     </visual>
   </link>
+    <!-- Left Wheel -->
+    <link name="left_wheel">
+      <collision>
+        <geometry>
+          <cylinder length="0.05" radius="0.1"/>
+        </geometry>
+        <origin xyz="0 0 0" rpy="0 1.5707 1.5707"/>
+      </collision>
+      <visual>
+        <geometry>
+          <cylinder length="0.05" radius="0.1"/>
+        </geometry>
+        <origin xyz="0 0 0" rpy="0 1.5707 1.5707"/>
+      </visual>
+      <inertial>
+        <mass value="5"/>
+        <inertia ixx="0.1" ixy="0" ixz="0" iyy="0.1" iyz="0" izz="0.1"/>
+        <origin xyz="0 0 0" rpy="0 1.5707 1.5707"/>
+      </inertial>
+    </link>
+    <!-- Right Wheel -->
+    <link name="right_wheel">
+      <collision>
+        <geometry>
+          <cylinder length="0.05" radius="0.1"/>
+        </geometry>
+        <origin xyz="0 0 0" rpy="0 1.5707 1.5707"/>
+      </collision>
+      <visual>
+        <geometry>
+          <cylinder length="0.05" radius="0.1"/>
+        </geometry>
+        <origin xyz="0 0 0" rpy="0 1.5707 1.5707"/>
+      </visual>
+      <inertial>
+        <mass value="5"/>
+        <inertia ixx="0.1" ixy="0" ixz="0" iyy="0.1" iyz="0" izz="0.1"/>
+        <origin xyz="0 0 0" rpy="0 1.5707 1.5707"/>
+      </inertial>
+    </link>
+  <joint type="continuous" name="left_wheel_hinge">
+    <origin xyz="0 0.15 0" rpy="0 0 0"/>
+    <child link="left_wheel"/>
+    <parent link="chassis"/>
+    <axis xyz="0 1 0" rpy="0 0 0"/>
+    <limit effort="10000" velocity="1000"/>
+    <dynamics damping="1.0" friction="1.0"/>
+  </joint>
+    <joint type="continuous" name="right_wheel_hinge">
+    <origin xyz="0 0.15 0" rpy="0 0 0"/>
+    <child link="right_wheel"/>
+    <parent link="chassis"/>
+    <axis xyz="0 1 0" rpy="0 0 0"/>
+    <limit effort="10000" velocity="1000"/>
+    <dynamics damping="1.0" friction="1.0"/>
+  </joint>
 </robot>

Commit message: add wheels

File: Project2/catkin_ws/src/my_robot/urdf/my_robot.xacro (robot description, xacro)
@@ -101,12 +101,11 @@
     <limit effort="10000" velocity="1000"/>
     <dynamics damping="1.0" friction="1.0"/>
-  </joint>
     <joint type="continuous" name="right_wheel_hinge">
-    <origin xyz="0 0.15 0" rpy="0 0 0"/>
-    <child link="right_wheel"/>
-    <parent link="chassis"/>
-    <axis xyz="0 1 0" rpy="0 0 0"/>
-    <limit effort="10000" velocity="1000"/>
-    <dynamics damping="1.0" friction="1.0"/>
-  </joint>
+      <origin xyz="0 -0.15 0" rpy="0 0 0"/>
+      <parent link="chassis"/>
+      <child link="right_wheel"/>
+      <axis xyz="0 1 0"/>
+      <limit effort="10000" velocity="1000"/>
+      <dynamics damping="1.0" friction="1.0"/>
+    </joint>
 </robot>

Commit message: add wheels

File: Project2/catkin_ws/src/my_robot/urdf/my_robot.xacro (robot description, xacro)
@@ -94,5 +94,5 @@
       </inertial>
     </link>
-  <joint type="continuous" name="left_wheel_hinge">
+    <joint type="continuous" name="left_wheel_hinge">
     <origin xyz="0 0.15 0" rpy="0 0 0"/>
     <child link="left_wheel"/>
@@ -101,4 +101,5 @@
     <limit effort="10000" velocity="1000"/>
     <dynamics damping="1.0" friction="1.0"/>
+    </joint>
     <joint type="continuous" name="right_wheel_hinge">
       <origin xyz="0 -0.15 0" rpy="0 0 0"/>

Commit message: add body color

File: Project2/catkin_ws/src/my_robot/urdf/my_robot.xacro (robot description, xacro)
@@ -28,4 +28,7 @@
         <box size=".4 .2 .1"/>
       </geometry>
+      <material name="red">
+        <color rgba="1 0 0 1"/>
+      </material>
     </visual>
     <collision name='back_caster_collision'>

Commit message: add mesh

File: Project2/catkin_ws/src/my_robot/urdf/my_robot.xacro (robot description, xacro)
@@ -27,4 +27,5 @@
       <geometry>
         <box size=".4 .2 .1"/>
+        <mesh filename="package://pr2_description/meshes/base_v0/base.dae"/>
       </geometry>
       <material name="red">

Commit message: add mesh

File: Project2/catkin_ws/src/my_robot/urdf/my_robot.xacro (robot description, xacro)
@@ -27,5 +27,4 @@
       <geometry>
         <box size=".4 .2 .1"/>
-        <mesh filename="package://pr2_description/meshes/base_v0/base.dae"/>
       </geometry>
       <material name="red">
@@ -114,3 +113,12 @@
       <dynamics damping="1.0" friction="1.0"/>
     </joint>
+    <gazebo reference="left_wheel">
+      <material>Gazebo/Yellow</material>
+    </gazebo>
+    <gazebo reference="right_wheel">
+      <material>Gazebo/Yellow</material>
+    </gazebo>
+    <gazebo reference="chassis">
+      <material>Gazebo/Green</material>
+    </gazebo>
 </robot>

Commit message: add camera and lidar

File: Project2/catkin_ws/src/my_robot/urdf/my_robot.xacro (robot description, xacro)
@@ -1,124 +1,178 @@
 <robot name="my_robot" xmlns:xacro="http://www.ros.org/wiki/xacro">
-  <link name="robot_footprint"></link>
-  <joint name="robot_footprint_joint" type="fixed">
-    <origin xyz="0 0 0" rpy="0 0 0" />
-    <parent link="robot_footprint"/>
-    <child link="chassis" />
-  </joint>
-  <link name='chassis'>
-    <pose>0 0 0.1 0 0 0</pose>
-    <inertial>
-      <mass value="15.0"/>
-      <origin xyz="0.0 0 0" rpy=" 0 0 0"/>
-      <inertia
-          ixx="0.1" ixy="0" ixz="0"
-          iyy="0.1" iyz="0"
-          izz="0.1"
-      />
-    </inertial>
-    <collision name='collision'>
-      <origin xyz="0 0 0" rpy=" 0 0 0"/>
-      <geometry>
-        <box size=".4 .2 .1"/>
-      </geometry>
-    </collision>
-    <visual name='chassis_visual'>
-      <origin xyz="0 0 0" rpy=" 0 0 0"/>
-      <geometry>
-        <box size=".4 .2 .1"/>
-      </geometry>
-      <material name="red">
-        <color rgba="1 0 0 1"/>
-      </material>
-    </visual>
-    <collision name='back_caster_collision'>
-      <origin xyz="-0.15 0 -0.05" rpy=" 0 0 0"/>
-      <geometry>
-        <sphere radius="0.0499"/>
-      </geometry>
-    </collision>
-    <visual name='back_caster_visual'>
-      <origin xyz="-0.15 0 -0.05" rpy=" 0 0 0"/>
-      <geometry>
-        <sphere radius="0.05"/>
-      </geometry>
-    </visual>
-    <collision name='front_caster_collision'>
-      <origin xyz="0.15 0 -0.05" rpy=" 0 0 0"/>
-      <geometry>
-        <sphere radius="0.0499"/>
-      </geometry>
-    </collision>
-    <visual name='front_caster_visual'>
-      <origin xyz="0.15 0 -0.05" rpy=" 0 0 0"/>
-      <geometry>
-        <sphere radius="0.05"/>
-      </geometry>
-    </visual>
-  </link>
+    <link name="robot_footprint"></link>
+    <joint name="robot_footprint_joint" type="fixed">
+        <origin xyz="0 0 0" rpy="0 0 0"/>
+        <parent link="robot_footprint"/>
+        <child link="chassis"/>
+    </joint>
+    <link name='chassis'>
+        <pose>0 0 0.1 0 0 0</pose>
+        <inertial>
+            <mass value="15.0"/>
+            <origin xyz="0.0 0 0" rpy=" 0 0 0"/>
+            <inertia
+                    ixx="0.1" ixy="0" ixz="0"
+                    iyy="0.1" iyz="0"
+                    izz="0.1"
+            />
+        </inertial>
+        <collision name='collision'>
+            <origin xyz="0 0 0" rpy=" 0 0 0"/>
+            <geometry>
+                <box size=".4 .2 .1"/>
+            </geometry>
+        </collision>
+        <visual name='chassis_visual'>
+            <origin xyz="0 0 0" rpy=" 0 0 0"/>
+            <geometry>
+                <box size=".4 .2 .1"/>
+            </geometry>
+            <material name="red">
+                <color rgba="1 0 0 1"/>
+            </material>
+        </visual>
+        <collision name='back_caster_collision'>
+            <origin xyz="-0.15 0 -0.05" rpy=" 0 0 0"/>
+            <geometry>
+                <sphere radius="0.0499"/>
+            </geometry>
+        </collision>
+        <visual name='back_caster_visual'>
+            <origin xyz="-0.15 0 -0.05" rpy=" 0 0 0"/>
+            <geometry>
+                <sphere radius="0.05"/>
+            </geometry>
+        </visual>
+        <collision name='front_caster_collision'>
+            <origin xyz="0.15 0 -0.05" rpy=" 0 0 0"/>
+            <geometry>
+                <sphere radius="0.0499"/>
+            </geometry>
+        </collision>
+        <visual name='front_caster_visual'>
+            <origin xyz="0.15 0 -0.05" rpy=" 0 0 0"/>
+            <geometry>
+                <sphere radius="0.05"/>
+            </geometry>
+        </visual>
+    </link>
     <!-- Left Wheel -->
     <link name="left_wheel">
-      <collision>
-        <geometry>
-          <cylinder length="0.05" radius="0.1"/>
-        </geometry>
-        <origin xyz="0 0 0" rpy="0 1.5707 1.5707"/>
-      </collision>
-      <visual>
-        <geometry>
-          <cylinder length="0.05" radius="0.1"/>
-        </geometry>
-        <origin xyz="0 0 0" rpy="0 1.5707 1.5707"/>
-      </visual>
-      <inertial>
-        <mass value="5"/>
-        <inertia ixx="0.1" ixy="0" ixz="0" iyy="0.1" iyz="0" izz="0.1"/>
-        <origin xyz="0 0 0" rpy="0 1.5707 1.5707"/>
-      </inertial>
+        <collision>
+            <geometry>
+                <cylinder length="0.05" radius="0.1"/>
+            </geometry>
+            <origin xyz="0 0 0" rpy="0 1.5707 1.5707"/>
+        </collision>
+        <visual>
+            <geometry>
+                <cylinder length="0.05" radius="0.1"/>
+            </geometry>
+            <origin xyz="0 0 0" rpy="0 1.5707 1.5707"/>
+        </visual>
+        <inertial>
+            <mass value="5"/>
+            <inertia ixx="0.1" ixy="0" ixz="0" iyy="0.1" iyz="0" izz="0.1"/>
+            <origin xyz="0 0 0" rpy="0 1.5707 1.5707"/>
+        </inertial>
     </link>
     <!-- Right Wheel -->
     <link name="right_wheel">
-      <collision>
-        <geometry>
-          <cylinder length="0.05" radius="0.1"/>
-        </geometry>
-        <origin xyz="0 0 0" rpy="0 1.5707 1.5707"/>
-      </collision>
-      <visual>
-        <geometry>
-          <cylinder length="0.05" radius="0.1"/>
-        </geometry>
-        <origin xyz="0 0 0" rpy="0 1.5707 1.5707"/>
-      </visual>
-      <inertial>
-        <mass value="5"/>
-        <inertia ixx="0.1" ixy="0" ixz="0" iyy="0.1" iyz="0" izz="0.1"/>
-        <origin xyz="0 0 0" rpy="0 1.5707 1.5707"/>
-      </inertial>
+        <collision>
+            <geometry>
+                <cylinder length="0.05" radius="0.1"/>
+            </geometry>
+            <origin xyz="0 0 0" rpy="0 1.5707 1.5707"/>
+        </collision>
+        <visual>
+            <geometry>
+                <cylinder length="0.05" radius="0.1"/>
+            </geometry>
+            <origin xyz="0 0 0" rpy="0 1.5707 1.5707"/>
+        </visual>
+        <inertial>
+            <mass value="5"/>
+            <inertia ixx="0.1" ixy="0" ixz="0" iyy="0.1" iyz="0" izz="0.1"/>
+            <origin xyz="0 0 0" rpy="0 1.5707 1.5707"/>
+        </inertial>
     </link>
     <joint type="continuous" name="left_wheel_hinge">
-    <origin xyz="0 0.15 0" rpy="0 0 0"/>
-    <child link="left_wheel"/>
-    <parent link="chassis"/>
-    <axis xyz="0 1 0" rpy="0 0 0"/>
-    <limit effort="10000" velocity="1000"/>
-    <dynamics damping="1.0" friction="1.0"/>
+        <origin xyz="0 0.15 0" rpy="0 0 0"/>
+        <child link="left_wheel"/>
+        <parent link="chassis"/>
+        <axis xyz="0 1 0" rpy="0 0 0"/>
+        <limit effort="10000" velocity="1000"/>
+        <dynamics damping="1.0" friction="1.0"/>
     </joint>
     <joint type="continuous" name="right_wheel_hinge">
-      <origin xyz="0 -0.15 0" rpy="0 0 0"/>
-      <parent link="chassis"/>
-      <child link="right_wheel"/>
-      <axis xyz="0 1 0"/>
-      <limit effort="10000" velocity="1000"/>
-      <dynamics damping="1.0" friction="1.0"/>
+        <origin xyz="0 -0.15 0" rpy="0 0 0"/>
+        <parent link="chassis"/>
+        <child link="right_wheel"/>
+        <axis xyz="0 1 0"/>
+        <limit effort="10000" velocity="1000"/>
+        <dynamics damping="1.0" friction="1.0"/>
+    </joint>
+    <!-- Camera Link -->
+    <link name="camera">
+        <visual>
+            <origin xyz="0 0 0" rpy="0 0 0"/>
+            <geometry>
+                <box size="0.05 0.05 0.05"/>
+            </geometry>
+        </visual>
+        <collision>
+            <origin xyz="0 0 0" rpy="0 0 0"/>
+            <geometry>
+                <box size="0.05 0.05 0.05"/>
+            </geometry>
+        </collision>
+        <inertial>
+            <origin xyz="0 0 0" rpy="0 0 0"/>
+            <mass value="0.1"/>
+            <inertia ixx="1e-6" ixy="0" ixz="0" iyy="1e-6" iyz="0" izz="1e-6"/>
+        </inertial>
+    </link>
+    <!-- Fixed Joint for Camera -->
+    <joint name="camera_joint" type="fixed">
+        <origin xyz="0.2 0 0" rpy="0 0 0"/>
+        <parent link="chassis"/>
+        <child link="camera"/>
+        <axis xyz="0 1 0"/>
+    </joint>
+    <!-- Hokuyo LIDAR Sensor Link -->
+    <link name="hokuyo">
+        <visual>
+            <origin xyz="0 0 0" rpy="0 0 0"/>
+            <geometry>
+                <mesh filename="package://my_robot/meshes/hokuyo.dae"/>
+            </geometry>
+        </visual>
+        <collision>
+            <origin xyz="0 0 0" rpy="0 0 0"/>
+            <geometry>
+                <box size="0.1 0.1 0.1"/>
+            </geometry>
+        </collision>
+        <inertial>
+            <origin xyz="0 0 0" rpy="0 0 0"/>
+            <mass value="1e-5"/>
+            <inertia ixx="1e-6" ixy="0" ixz="0" iyy="1e-6" iyz="0" izz="1e-6"/>
+        </inertial>
+    </link>
+    <!-- Fixed Joint for Hokuyo -->
+    <joint name="hokuyo_joint" type="fixed">
+        <origin xyz="0.15 0 0.1" rpy="0 0 0"/>
+        <parent link="chassis"/>
+        <child link="hokuyo"/>
+        <axis xyz="0 1 0"/>
     </joint>
     <gazebo reference="left_wheel">
-      <material>Gazebo/Yellow</material>
+        <material>Gazebo/Yellow</material>
     </gazebo>
     <gazebo reference="right_wheel">
-      <material>Gazebo/Yellow</material>
+        <material>Gazebo/Yellow</material>
     </gazebo>
     <gazebo reference="chassis">
-      <material>Gazebo/Green</material>
+        <material>Gazebo/Green</material>
     </gazebo>
 </robot>

Commit message: add camera and lidar

File: Project2/catkin_ws/src/my_robot/urdf/my_robot.xacro (robot description, xacro)
@@ -176,3 +176,9 @@
         <material>Gazebo/Green</material>
     </gazebo>
+    <gazebo reference="hokuyo">
+        <material>Gazebo/Red</material>
+    </gazebo>
+        <gazebo reference="camera">
+        <material>Gazebo/Blue</material>
+    </gazebo>
 </robot>
