Commit message: rework

File: Project4/catkin_ws/src/my_robot/urdf/my_robot.xacro (robot description, xacro)
@@ -142,4 +142,11 @@
         <axis xyz="0 1 0"/>
     </joint>
+    <joint name="camera_optical_joint" type="fixed">
+        <origin xyz="0 0 0" rpy="-1.5707 0 -1.5707"/>
+        <parent link="camera_link"/>
+        <child link="camera_link_optical"/>
+    </joint>
+    <link name="camera_link_optical">
+    </link>
     <!-- Hokuyo LIDAR Sensor Link -->
     <link name="hokuyo">
